File: Electronics/DATA/MANTA.kicad_sch (KiCad schematic)
At the start: 37 parts, among them J1 LORA_UP, J2 LORA_DOWN

Commit message: final pcb boards design
Parts:
- removed Battery_4S1: Conn_01x02, Connector_AMASS:AMASS_XT60PW-M_1x02_P7.20mm_Horizontal, symbol Connector_Generic:Conn_01x02
- removed ESC_INPUT1: (no value), Connector_Wire:SolderWire-2.5sqmm_1x02_P8.8mm_D2.4mm_OD4.4mm, symbol Connector_Generic:Conn_01x02
- removed ESC_OUT_+_S1, RASP_UART1, RECEIVER_POWER1, SERVO_BL1, SERVO_BR1, SERVO_FL1, SERVO_FR1, VOLTAGE_SENSOR_DATA1: Conn_01x03, Connector_PinHeader_2.54mm:PinHeader_1x03_P2.54mm_Vertical, symbol Connector_Generic:Conn_01x03
- removed EXTRA_ENERGY_15V1, EXTRA_ENERGY_5V1, RASP_POWER1: Conn_01x02, Connector_PinHeader_2.54mm:PinHeader_1x02_P2.54mm_Vertical, symbol Connector_Generic:Conn_01x02
- removed Stepdown_IN_+1, Stepdown_IN_+2, Stepdown_IN_-1, Stepdown_IN_-2, Stepdown_OUT_+1, Stepdown_OUT_+2, Stepdown_OUT_-1, Stepdown_OUT_-2: Conn_01x01, Connector_PinHeader_2.54mm:PinHeader_1x01_P2.54mm_Vertical, symbol Connector_Generic:Conn_01x01
- removed VOLTAGE_SENSOR_IN1: (no value), Connector_PinHeader_2.54mm:PinHeader_1x02_P2.54mm_Vertical, symbol Connector_Generic:Conn_01x02
- added CORNER_3V1, CORNER_3V2, CORNER_GND1, CORNER_GND2: Conn_01x06, Connector_PinHeader_2.54mm:PinHeader_1x06_P2.54mm_Vertical, symbol Connector_Generic:Conn_01x06
- added DATA_BRIDGE1: Conn_01x08, Connector_PinHeader_2.54mm:PinHeader_1x08_P2.54mm_Vertical, symbol Connector_Generic:Conn_01x08
- added I2C_RASP1: Conn_01x03, Connector_PinHeader_2.54mm:PinHeader_1x03_P2.54mm_Vertical, symbol Connector_Generic:Conn_01x03
- added R10, R11, R12, R7, R8, R9: 2k, Resistor_THT:R_Axial_DIN0207_L6.3mm_D2.5mm_P10.16mm_Horizontal, symbol Device:R
- added R13, R14: 10k, Resistor_THT:R_Axial_DIN0207_L6.3mm_D2.5mm_P10.16mm_Horizontal, symbol Device:R
- added R6: 1k, Resistor_THT:R_Axial_DIN0207_L6.3mm_D2.5mm_P10.16mm_Horizontal, symbol Device:R
Connections:
- net +3.3V: now also CORNER_3V1.1 (Pin_1), CORNER_3V1.2 (Pin_2), CORNER_3V1.3 (Pin_3), CORNER_3V1.4 (Pin_4), CORNER_3V1.5 (Pin_5), CORNER_3V1.6 (Pin_6), CORNER_3V2.1 (Pin_1), CORNER_3V2.2 (Pin_2), CORNER_3V2.3 (Pin_3), CORNER_3V2.4 (Pin_4), CORNER_3V2.5 (Pin_5), CORNER_3V2.6 (Pin_6), R13.1, R14.1
- net BATTERY_DATA: now also DATA_BRIDGE1.2 (Pin_2)
- net CH1_INPUT: now also R7.2
- net CH2_INPUT: now also R8.2
- net CH3_INPUT: now also R9.2
- net CH4_INPUT: now also R10.2
- net CH5_INPUT: now also R11.2
- net ESC_THROTTLE: now also DATA_BRIDGE1.3 (Pin_3)
- net GND: now also CORNER_GND1.1 (Pin_1), CORNER_GND1.2 (Pin_2), CORNER_GND1.3 (Pin_3), CORNER_GND1.4 (Pin_4), CORNER_GND1.5 (Pin_5), CORNER_GND1.6 (Pin_6), CORNER_GND2.1 (Pin_1), CORNER_GND2.2 (Pin_2), CORNER_GND2.3 (Pin_3), CORNER_GND2.4 (Pin_4), CORNER_GND2.5 (Pin_5), CORNER_GND2.6 (Pin_6), DATA_BRIDGE1.8 (Pin_8), I2C_RASP1.1 (Pin_1), R10.1, R11.1, R12.1, R7.1, R8.1, R9.1
- net I2C_SCL: now also I2C_EXTRA_1.3 (Pin_3), I2C_EXTRA_2.3 (Pin_3), I2C_RASP1.2 (Pin_2), R13.2; no longer I2C_EXTRA_1.4 (Pin_4), I2C_EXTRA_2.4 (Pin_4)
- net I2C_SDA: now also I2C_EXTRA_1.4 (Pin_4), I2C_EXTRA_2.4 (Pin_4), I2C_RASP1.3 (Pin_3), R14.2; no longer I2C_EXTRA_1.3 (Pin_3), I2C_EXTRA_2.3 (Pin_3)
- net SERVO_BL_CTRL: now also DATA_BRIDGE1.7 (Pin_7)
- net SERVO_BR_CTRL: now also DATA_BRIDGE1.4 (Pin_4)
- net SERVO_FL_CTRL: now also DATA_BRIDGE1.6 (Pin_6)
- net SERVO_FR_CTRL: now also DATA_BRIDGE1.5 (Pin_5)
- net at RECEIVER_SIGNALS1.6 (Pin_6): now also R6.2
- net UART_ESP_RX: no longer names the net of ESP32-RIGHT1.4 (Pin_4)
- net UART_ESP_TX: no longer names the net of ESP32-RIGHT1.3 (Pin_3)
- new net CH6_INPUT: DATA_BRIDGE1.1 (Pin_1), R12.2, R6.1
- no-connect marks 20 -> 19
Other:
- title: MAIN PCB -> LOGIC PCB
- moved on the sheet: Barometer_BMP280, GPS1, MPU6050_GYRO_ACC1, RECEIVER_SIGNALS1
