File: Electronics/DATA/MANTA.kicad_pcb (KiCad board)
At the start: 4 copper layers, 41 parts, among them J1 LORA_UP, J2 LORA_DOWN

Commit message: final pcb boards design
Parts:
- removed Battery_4S1: Conn_01x02, Connector_AMASS:AMASS_XT60PW-M_1x02_P7.20mm_Horizontal
- removed ESC_BEC1, EXTRA_ENERGY_15V1, EXTRA_ENERGY_5V1, RASP_POWER1, RECEIVER_POWER1, UBEC_IN1, UBEC_OUT1: Conn_01x02, Connector_PinHeader_2.54mm:PinHeader_1x02_P2.54mm_Vertical
- removed ESC_INPUT1: ~, Connector_Wire:SolderWire-2.5sqmm_1x02_P8.8mm_D2.4mm_OD4.4mm
- removed ESC_OUT_+_S1, RASP_UART1, RECEIVER_POWER1, SERVO_BL1, SERVO_BR1, SERVO_FL1, SERVO_FR1, VOLTAGE_SENSOR_DATA1: Conn_01x03, Connector_PinHeader_2.54mm:PinHeader_1x03_P2.54mm_Vertical
- removed Stepdown_IN_+1, Stepdown_IN_+2, Stepdown_IN_-1, Stepdown_IN_-2, Stepdown_OUT_+1, Stepdown_OUT_+2, Stepdown_OUT_-1, Stepdown_OUT_-2: Conn_01x01, Connector_PinHeader_2.54mm:PinHeader_1x01_P2.54mm_Vertical
- removed VOLTAGE_SENSOR_IN1: ~, Connector_PinHeader_2.54mm:PinHeader_1x02_P2.54mm_Vertical
- added CORNER_3V1: Conn_01x06, Connector_PinHeader_2.54mm:PinHeader_1x06_P2.54mm_Vertical, F.Cu at (59.0, 3.00)
- added CORNER_3V2: Conn_01x06, Connector_PinHeader_2.54mm:PinHeader_1x06_P2.54mm_Vertical, F.Cu at (2.00, 97.0)
- added CORNER_GND1: Conn_01x06, Connector_PinHeader_2.54mm:PinHeader_1x06_P2.54mm_Vertical, F.Cu at (2.00, 3.00)
- added CORNER_GND2: Conn_01x06, Connector_PinHeader_2.54mm:PinHeader_1x06_P2.54mm_Vertical, F.Cu at (59.0, 97.0)
- added DATA_BRIDGE1: Conn_01x08, Connector_PinHeader_2.54mm:PinHeader_1x08_P2.54mm_Vertical, F.Cu at (58.0, 61.0)
- added I2C_RASP1: Conn_01x03, Connector_PinHeader_2.54mm:PinHeader_1x03_P2.54mm_Vertical, F.Cu at (27.7, 2.54)
- added R10: 2k, Resistor_THT:R_Axial_DIN0207_L6.3mm_D2.5mm_P10.16mm_Horizontal, F.Cu at (42.7, 49.0)
- added R11: 2k, Resistor_THT:R_Axial_DIN0207_L6.3mm_D2.5mm_P10.16mm_Horizontal, F.Cu at (45.7, 49.0)
- added R12: 2k, Resistor_THT:R_Axial_DIN0207_L6.3mm_D2.5mm_P10.16mm_Horizontal, F.Cu at (48.8, 49.0)
- added R13: 10k, Resistor_THT:R_Axial_DIN0207_L6.3mm_D2.5mm_P10.16mm_Horizontal, F.Cu at (54.6, 92.5)
- added R14: 10k, Resistor_THT:R_Axial_DIN0207_L6.3mm_D2.5mm_P10.16mm_Horizontal, F.Cu at (8.13, 65.0)
- added R6: 1k, Resistor_THT:R_Axial_DIN0207_L6.3mm_D2.5mm_P10.16mm_Horizontal, F.Cu at (49.0, 35.3)
- added R7: 2k, Resistor_THT:R_Axial_DIN0207_L6.3mm_D2.5mm_P10.16mm_Horizontal, F.Cu at (33.5, 49.0)
- added R8: 2k, Resistor_THT:R_Axial_DIN0207_L6.3mm_D2.5mm_P10.16mm_Horizontal, F.Cu at (36.6, 49.0)
- added R9: 2k, Resistor_THT:R_Axial_DIN0207_L6.3mm_D2.5mm_P10.16mm_Horizontal, F.Cu at (39.6, 49.0)
- moved I2C_EXTRA_2 269.5 mm to (11.9, 2.29), turned to 90 degrees
- moved J2 266.7 mm to (6.15, 9.40), turned to 90 degrees
- moved J1 252.9 mm to (6.15, 34.8), turned to 90 degrees
- moved I2C_EXTRA_1 244.4 mm to (2.00, 66.0)
- moved GPS1 220.8 mm to (15.2, 98.0), turned to 90 degrees
- moved ESP32-RIGHT1 103.6 mm to (28.1, 20.2), turned to 0 degrees
- moved ESP32-LEFT1 101.3 mm to (53.5, 55.8), turned to 180 degrees
- moved Barometer_BMP280 84.0 mm to (20.8, 43.5), turned to -90 degrees
- moved RECEIVER_SIGNALS1 64.1 mm to (38.6, 2.00)
- moved R1 58.9 mm to (33.5, 35.3)
- moved R2 56.9 mm to (36.6, 35.3)
- moved R3 54.9 mm to (39.6, 35.3)
- moved R4 52.8 mm to (42.7, 35.3)
- moved R5 50.8 mm to (45.7, 35.3)
- moved MPU6050_GYRO_ACC1 31.4 mm to (53.8, 98.0), turned to -90 degrees
Connections:
- ESP32-RIGHT1 pad 3: /UART_ESP_TX -> unconnected-(ESP32-RIGHT1-Pin_3-Pad3)
- ESP32-RIGHT1 pad 4: /UART_ESP_RX -> unconnected-(ESP32-RIGHT1-Pin_4-Pad4)
- I2C_EXTRA_1 pad 3: /I2C_SDA -> /I2C_SCL
- I2C_EXTRA_1 pad 4: /I2C_SCL -> /I2C_SDA
- I2C_EXTRA_2 pad 3: /I2C_SDA -> /I2C_SCL
- I2C_EXTRA_2 pad 4: /I2C_SCL -> /I2C_SDA
- RECEIVER_SIGNALS1 pad 6: unconnected-(RECEIVER_SIGNALS1-Pin_6-Pad6) -> Net-(RECEIVER_SIGNALS1-Pin_6)
Routing:
- net +3.3V: track 0.00 -> 395.6 mm
- net /I2C_SDA: track 0.00 -> 256.1 mm
- net /I2C_SCL: track 0.00 -> 213.1 mm
- net /GPS_TX: track 0.00 -> 73.8 mm
- net /SERVO_BL_CTRL: track 0.00 -> 72.4 mm
- net /SERVO_FL_CTRL: track 0.00 -> 72.3 mm
- net /GPS_RX: track 0.00 -> 72.0 mm
- net /SERVO_FR_CTRL: track 0.00 -> 62.1 mm
- net /SERVO_BR_CTRL: track 0.00 -> 46.5 mm
- net /SPI_MOSI: track 0.00 -> 38.2 mm
- net /CH6_INPUT: track 0.00 -> 33.3 mm
- net /ESC_THROTTLE: track 0.00 -> 31.7 mm
- net /SPI_DI0_LORA: track 0.00 -> 28.8 mm
- net /CH1_INPUT: track 0.00 -> 28.4 mm
- net Net-(RECEIVER_SIGNALS1-Pin_1): track 0.00 -> 25.2 mm
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- added copper zone on B.Cu, net GND
Other:
- board outline added: 61 x 100 mm
- copper layers 4 -> 2
- board text added: "Afonso Nóia"
- board text added: "BAROMETER"
- board text added: "DATA BRIDGE"
- board text added: "ESP32"
- board text added: "GPS"
- board text added: "I2C EXTRA"
- board text added: "I2C EXTRA 1"
- board text added: "I2C RASP"
- board text added: "IMU"
- board text added: "LoRa"
- board text added: "MANTA"
- board text added: "RECEIVER"
- board text added: "[A]"
- board text added: "[USB]"

Commit message: feat: flight validation with calibrated PIDs, Raspberry Pi onboard recording and restructured documentation
- Restructure README.md showcasing flight test validation, calibrated PIDs, and companion computer video pipeline
- Add clickable onboard flight video banner linking to YouTube footage starting at 1:30 min
- Add optimized pre-flight field inspection photo and physical assembled electronics stack
- Document PI-D closed-loop control, surface trims, flaperons governor (20 deg down) with anti-saturation headroom scaling
- Document Raspberry Pi 3 A+ autonomous boot stack, RF cutoff, and power-loss-immune MKV recording
- Add Ground Station flight replay simulator and GPS auto-pin probing
- Update roadmap marking Phases 1, 2, and 3 100% completed with all 171 CI/CD tests passing
Other:
- board text added: "Afonso Noia"
- board text removed: "Afonso Nóia"
Changed lines of the file:
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@@
 		)
 	)
-	(gr_text "Afonso Nóia"
+	(gr_text "Afonso Noia"
 		(at 30.5 76.5 0)
 		(layer "F.SilkS")
