File: Electronics/POWER/MANTA.kicad_sch (KiCad schematic)
At the start: 19 parts

Commit message: final pcb boards design
Parts:
- removed CORNER_3V_1, CORNER_3V_2, CORNER_GND_1, CORNER_GND_2: Conn_01x03, Connector_PinHeader_2.54mm:PinHeader_1x03_P2.54mm_Vertical, symbol Connector_Generic:Conn_01x03
- removed Stepdown_IN_+1, Stepdown_IN_+2, Stepdown_IN_-1, Stepdown_IN_-2, Stepdown_OUT_+1, Stepdown_OUT_+2, Stepdown_OUT_-1, Stepdown_OUT_-2: Conn_01x01, Connector_PinHeader_2.54mm:PinHeader_1x01_P2.54mm_Vertical, symbol Connector_Generic:Conn_01x01
- added CH6_PIN1, Stepdown_IN_+1, Stepdown_IN_+2, Stepdown_IN_-1, Stepdown_IN_-2, Stepdown_OUT_+1, Stepdown_OUT_+2, Stepdown_OUT_-1, Stepdown_OUT_-2: Conn_01x02, Connector_PinHeader_2.54mm:PinHeader_1x02_P2.54mm_Vertical, symbol Connector_Generic:Conn_01x02
- added CORNER_3V_1, CORNER_3V_2, CORNER_GND_1, CORNER_GND_2: Conn_01x06, Connector_PinHeader_2.54mm:PinHeader_1x06_P2.54mm_Vertical, symbol Connector_Generic:Conn_01x06
- added DATA_BRIDGE1: Conn_01x08, Connector_PinHeader_2.54mm:PinHeader_1x08_P2.54mm_Vertical, symbol Connector_Generic:Conn_01x08
- added ESC_IN_UBEC1, SERVO_BL1, SERVO_BR1, SERVO_FL1, SERVO_FR1, VOLTAGE_SENSOR_DATA1: Conn_01x03, Connector_PinHeader_2.54mm:PinHeader_1x03_P2.54mm_Vertical, symbol Connector_Generic:Conn_01x03
Connections:
- net +15V: now also Battery_4S1.2 (Pin_2), Stepdown_IN_+1.1 (Pin_1), Stepdown_IN_+1.2 (Pin_2), Stepdown_IN_+2.1 (Pin_1), Stepdown_IN_+2.2 (Pin_2); no longer Battery_4S1.1 (Pin_1)
- net +3.3V: now also CORNER_3V_1.1 (Pin_1), CORNER_3V_1.2 (Pin_2), CORNER_3V_1.3 (Pin_3), CORNER_3V_1.4 (Pin_4), CORNER_3V_1.5 (Pin_5), CORNER_3V_1.6 (Pin_6), CORNER_3V_2.1 (Pin_1), CORNER_3V_2.2 (Pin_2), CORNER_3V_2.3 (Pin_3), CORNER_3V_2.4 (Pin_4), CORNER_3V_2.5 (Pin_5), CORNER_3V_2.6 (Pin_6), Stepdown_OUT_+1.1 (Pin_1), Stepdown_OUT_+1.2 (Pin_2)
- net +5VA: now also Stepdown_OUT_+2.1 (Pin_1), Stepdown_OUT_+2.2 (Pin_2)
- net GND: now also Battery_4S1.1 (Pin_1), CORNER_GND_1.1 (Pin_1), CORNER_GND_1.2 (Pin_2), CORNER_GND_1.3 (Pin_3), CORNER_GND_1.4 (Pin_4), CORNER_GND_1.5 (Pin_5), CORNER_GND_1.6 (Pin_6), CORNER_GND_2.1 (Pin_1), CORNER_GND_2.2 (Pin_2), CORNER_GND_2.3 (Pin_3), CORNER_GND_2.4 (Pin_4), CORNER_GND_2.5 (Pin_5), CORNER_GND_2.6 (Pin_6), DATA_BRIDGE1.8 (Pin_8), ESC_IN_UBEC1.3 (Pin_3), SERVO_BL1.3 (Pin_3), SERVO_BR1.3 (Pin_3), SERVO_FL1.3 (Pin_3), SERVO_FR1.3 (Pin_3), Stepdown_IN_-1.1 (Pin_1), Stepdown_IN_-1.2 (Pin_2), Stepdown_IN_-2.1 (Pin_1), Stepdown_IN_-2.2 (Pin_2), Stepdown_OUT_-1.1 (Pin_1), Stepdown_OUT_-1.2 (Pin_2), Stepdown_OUT_-2.1 (Pin_1), Stepdown_OUT_-2.2 (Pin_2), VOLTAGE_SENSOR_DATA1.3 (Pin_3); no longer Battery_4S1.2 (Pin_2)
- new net +5V: ESC_IN_UBEC1.2 (Pin_2), SERVO_BL1.2 (Pin_2), SERVO_BR1.2 (Pin_2), SERVO_FL1.2 (Pin_2), SERVO_FR1.2 (Pin_2)
- new net CH6_INPUT: CH6_PIN1.1 (Pin_1), CH6_PIN1.2 (Pin_2), DATA_BRIDGE1.1 (Pin_1)
- new net SIGNAL_THROTTLE: DATA_BRIDGE1.3 (Pin_3), ESC_IN_UBEC1.1 (Pin_1)
- new net S_SERVO_BL: DATA_BRIDGE1.7 (Pin_7), SERVO_BL1.1 (Pin_1)
- new net S_SERVO_BR: DATA_BRIDGE1.4 (Pin_4), SERVO_BR1.1 (Pin_1)
- new net S_SERVO_FL: DATA_BRIDGE1.6 (Pin_6), SERVO_FL1.1 (Pin_1)
- new net S_SERVO_FR: DATA_BRIDGE1.5 (Pin_5), SERVO_FR1.1 (Pin_1)
- new net VOLTAGE_DATA: DATA_BRIDGE1.2 (Pin_2), VOLTAGE_SENSOR_DATA1.1 (Pin_1)
- no-connect marks 1 -> 2
Other:
- moved on the sheet: VOLTAGE_SENSOR_IN1
