File: Electronics/POWER/MANTA.kicad_pcb (KiCad board)
At the start: 4 copper layers, 61 x 100 mm, 19 parts

Commit message: final pcb boards design
Parts:
- added CH6_PIN1: Conn_01x02, Connector_PinHeader_2.54mm:PinHeader_1x02_P2.54mm_Vertical, F.Cu at (49.3, 8.38)
- added DATA_BRIDGE1: Conn_01x08, Connector_PinHeader_2.54mm:PinHeader_1x08_P2.54mm_Vertical, B.Cu at (58.0, 61.0)
- added ESC_IN_UBEC1: Conn_01x03, Connector_PinHeader_2.54mm:PinHeader_1x03_P2.54mm_Vertical, F.Cu at (29.0, 33.0)
- added SERVO_BL1: Conn_01x03, Connector_PinHeader_2.54mm:PinHeader_1x03_P2.54mm_Vertical, F.Cu at (10.5, 27.5)
- added SERVO_BR1: Conn_01x03, Connector_PinHeader_2.54mm:PinHeader_1x03_P2.54mm_Vertical, F.Cu at (50.5, 27.5)
- added SERVO_FL1: Conn_01x03, Connector_PinHeader_2.54mm:PinHeader_1x03_P2.54mm_Vertical, F.Cu at (10.5, 18.0)
- added SERVO_FR1: Conn_01x03, Connector_PinHeader_2.54mm:PinHeader_1x03_P2.54mm_Vertical, F.Cu at (50.5, 18.0)
- added VOLTAGE_SENSOR_DATA1: Conn_01x03, Connector_PinHeader_2.54mm:PinHeader_1x03_P2.54mm_Vertical, B.Cu at (45.0, 90.7)
- CORNER_3V_1, CORNER_3V_2, CORNER_GND_1, CORNER_GND_2: value Conn_01x03 -> Conn_01x06; footprint Connector_PinHeader_2.54mm:PinHeader_1x03_P2.54mm_Vertical -> Connector_PinHeader_2.54mm:PinHeader_1x06_P2.54mm_Vertical; moved to B.Cu
- Stepdown_IN_+1, Stepdown_IN_+2, Stepdown_IN_-1, Stepdown_IN_-2, Stepdown_OUT_+1, Stepdown_OUT_+2, Stepdown_OUT_-1, Stepdown_OUT_-2: value Conn_01x01 -> Conn_01x02; footprint Connector_PinHeader_2.54mm:PinHeader_1x01_P2.54mm_Vertical -> Connector_PinHeader_2.54mm:PinHeader_1x02_P2.54mm_Vertical
- moved EXTRA_ENERGY_15V1 9.00 mm to (59.0, 24.0)
- moved EXTRA_ENERGY_5V1 9.00 mm to (2.00, 24.0)
- moved Stepdown_IN_-2 6.39 mm to (9.40, 62.2), turned to -90 degrees
- moved Stepdown_OUT_-2 6.39 mm to (49.4, 62.2), turned to 90 degrees
- moved Stepdown_IN_+2 6.10 mm to (9.40, 44.2), turned to -90 degrees
- moved Stepdown_OUT_+2 6.10 mm to (49.4, 44.2), turned to 90 degrees
- moved RECEIVER_POWER1 3.50 mm to (48.5, 2.00)
- moved Stepdown_OUT_-1 3.42 mm to (49.1, 86.8), turned to 90 degrees
- moved Stepdown_IN_-1 3.42 mm to (9.14, 86.8), turned to -90 degrees
- moved Stepdown_OUT_+1 3.18 mm to (49.1, 68.8), turned to 90 degrees
- moved Stepdown_IN_+1 3.18 mm to (9.14, 68.8), turned to -90 degrees
- moved VOLTAGE_SENSOR_IN1 1.47 mm to (46.2, 98.0)
- moved Battery_4S1 1.01 mm to (27.7, 8.50)
- moved ESC_INPUT1 0.34 mm to (27.2, 96.5)
- turned CORNER_3V_1 to 180 degrees
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Connections:
- Battery_4S1 pad 1: +15V -> GND
- Battery_4S1 pad 2: GND -> +15V
Routing:
- net /S_SERVO_FL: track 0.00 -> 88.1 mm
- net /S_SERVO_BL: track 0.00 -> 83.2 mm
- net /SIGNAL_THROTTLE: track 0.00 -> 77.7 mm
- net /CH6_INPUT: track 0.00 -> 66.1 mm
- net /S_SERVO_FR: track 0.00 -> 65.8 mm
- net /S_SERVO_BR: track 0.00 -> 56.4 mm
- net /VOLTAGE_DATA: track 0.00 -> 38.9 mm
- added copper zone on In1.Cu, net +15V
- added copper zone on In2.Cu, net +3.3V
- added copper zone on F.Cu, net +5V
- added copper zone on F.Cu, net +5VA
- added copper zone on B.Cu, net GND
- removed copper zone on In2.Cu, net +15V
- removed copper zone on F.Cu, net +3.3V
- removed copper zone on B.Cu, net +5VA
- removed copper zone on In1.Cu, net GND
Other:
- board text added: "BL"
- board text added: "BR"
- board text added: "CH6"
- board text added: "DATA BRIDGE"
- board text added: "ESC"
- board text added: "ESC UBEC"
- board text added: "FL"
- board text added: "FR"
- board text added: "RASPBERRY POWER"
- board text added: "RECEIVER"
- board text added: "S"
- board text added: "T"
- board text added: "VD"
- board text removed: "RASP_POWER"
- board text removed: "RECEIVER_POWER"

Commit message: feat: flight validation with calibrated PIDs, Raspberry Pi onboard recording and restructured documentation
- Restructure README.md showcasing flight test validation, calibrated PIDs, and companion computer video pipeline
- Add clickable onboard flight video banner linking to YouTube footage starting at 1:30 min
- Add optimized pre-flight field inspection photo and physical assembled electronics stack
- Document PI-D closed-loop control, surface trims, flaperons governor (20 deg down) with anti-saturation headroom scaling
- Document Raspberry Pi 3 A+ autonomous boot stack, RF cutoff, and power-loss-immune MKV recording
- Add Ground Station flight replay simulator and GPS auto-pin probing
- Update roadmap marking Phases 1, 2, and 3 100% completed with all 171 CI/CD tests passing
Other:
- board text added: "Afonso Noia"
- board text removed: "Afonso Nóia"
Changed lines of the file:
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@@
 		)
 	)
-	(gr_text "Afonso Nóia "
+	(gr_text "Afonso Noia "
 		(at 30.5 26 0)
 		(layer "F.SilkS")
